Commit message: Adição dos arquivos referentes ao robô lucasrobot

File: interbotix_ros_xsarms/interbotix_xsarm_descriptions/urdf/lucasrobot.urdf.xacro (robot description, xacro)
@@ -1,5 +1,5 @@
 <?xml version="1.0"?>
-<robot name="vx300s" xmlns:xacro="http://ros.org/wiki/xacro">
-  <xacro:arg name="robot_name" default = "vx300s"/>
+<robot name="lucasrobot" xmlns:xacro="http://ros.org/wiki/xacro">
+  <xacro:arg name="robot_name" default = "lucasrobot"/>
   <xacro:arg name="base_link_frame" default="base_link"/>
   <xacro:arg name="show_ar_tag" default="false"/>
@@ -26,14 +26,14 @@
   <link name="$(arg robot_name)/$(arg base_link_frame)">
     <visual>
-      <origin rpy="0 0 ${pi/2}" xyz="0 0 0"/>
-      <geometry>
-        <mesh filename="package://interbotix_xsarm_descriptions/meshes/vx300s_meshes/vx300s_1_base.stl" scale="0.001 0.001 0.001"/>
-      </geometry>
-      <material name="interbotix_black"/>
-    </visual>
-    <collision>
-      <origin rpy="0 0 ${pi/2}" xyz="0 0 0"/>
-      <geometry>
-        <mesh filename="package://interbotix_xsarm_descriptions/meshes/vx300s_meshes/vx300s_1_base.stl" scale="0.001 0.001 0.001"/>
+      <origin rpy="0 0 ${pi/2}" xyz="-0.045 0 0"/>
+      <geometry>
+        <mesh filename="package://interbotix_xsarm_descriptions/meshes/lucasrobot_meshes/lucasrobot_1_base.stl" scale="0.001 0.001 0.001"/>
+      </geometry>
+      <material name="interbotix_black"/>
+    </visual>
+    <collision>
+      <origin rpy="0 0 ${pi/2}" xyz="-0.045 0 0"/>
+      <geometry>
+        <mesh filename="package://interbotix_xsarm_descriptions/meshes/lucasrobot_meshes/lucasrobot_1_base.stl" scale="0.001 0.001 0.001"/>
       </geometry>
     </collision>
@@ -47,5 +47,5 @@
     <axis xyz="0 0 1"/>
     <limit effort="10" lower="${-pi + pi_offset}" upper="${pi - pi_offset}" velocity="${pi}"/>
-    <origin rpy="0 0 0" xyz="0 0 0.079"/>
+    <origin rpy="0 0 0" xyz="0 0 0.05"/>
     <parent link="$(arg robot_name)/$(arg base_link_frame)"/>
     <child link="$(arg robot_name)/shoulder_link"/>
@@ -63,14 +63,14 @@
   <link name="$(arg robot_name)/shoulder_link">
     <visual>
+      <origin rpy="0 0 ${pi/2}" xyz="0 0 0"/>
+      <geometry>
+        <mesh filename="package://interbotix_xsarm_descriptions/meshes/lucasrobot_meshes/lucasrobot_2_shoulder.stl" scale="0.001 0.001 0.001"/>
+      </geometry>
+      <material name="interbotix_black"/>
+    </visual>
+    <collision>
       <origin rpy="0 0 ${pi/2}" xyz="0 0 -0.003"/>
       <geometry>
-        <mesh filename="package://interbotix_xsarm_descriptions/meshes/vx300s_meshes/vx300s_2_shoulder.stl" scale="0.001 0.001 0.001"/>
-      </geometry>
-      <material name="interbotix_black"/>
-    </visual>
-    <collision>
-      <origin rpy="0 0 ${pi/2}" xyz="0 0 -0.003"/>
-      <geometry>
-        <mesh filename="package://interbotix_xsarm_descriptions/meshes/vx300s_meshes/vx300s_2_shoulder.stl" scale="0.001 0.001 0.001"/>
+        <mesh filename="package://interbotix_xsarm_descriptions/meshes/lucasrobot_meshes/lucasrobot_2_shoulder.stl" scale="0.001 0.001 0.001"/>
       </geometry>
     </collision>
@@ -84,5 +84,5 @@
     <axis xyz="0 1 0"/>
     <limit effort="20" lower="${radians(-106)}" upper="${radians(72)}" velocity="${pi}"/>
-    <origin rpy="0 0 0" xyz="0 0 0.04805"/>
+    <origin rpy="0 0 0" xyz="0 0 0.065"/>
     <parent link="$(arg robot_name)/shoulder_link"/>
     <child link="$(arg robot_name)/upper_arm_link"/>
@@ -100,14 +100,14 @@
   <link name="$(arg robot_name)/upper_arm_link">
     <visual>
+      <origin rpy="0 0 ${pi/2}" xyz="0.025 0 -0.013"/>
+      <geometry>
+        <mesh filename="package://interbotix_xsarm_descriptions/meshes/lucasrobot_meshes/lucasrobot_3_upper_arm.stl" scale="0.001 0.001 0.001"/>
+      </geometry>
+      <material name="interbotix_black"/>
+    </visual>
+    <collision>
       <origin rpy="0 0 ${pi/2}" xyz="0 0 0"/>
       <geometry>
-        <mesh filename="package://interbotix_xsarm_descriptions/meshes/vx300s_meshes/vx300s_3_upper_arm.stl" scale="0.001 0.001 0.001"/>
-      </geometry>
-      <material name="interbotix_black"/>
-    </visual>
-    <collision>
-      <origin rpy="0 0 ${pi/2}" xyz="0 0 0"/>
-      <geometry>
-        <mesh filename="package://interbotix_xsarm_descriptions/meshes/vx300s_meshes/vx300s_3_upper_arm.stl" scale="0.001 0.001 0.001"/>
+        <mesh filename="package://interbotix_xsarm_descriptions/meshes/lucasrobot_meshes/lucasrobot_3_upper_arm.stl" scale="0.001 0.001 0.001"/>
       </geometry>
     </collision>
@@ -121,7 +121,7 @@
     <axis xyz="0 1 0"/>
     <limit effort="15" lower="${radians(-101)}" upper="${radians(92)}" velocity="${pi}"/>
-    <origin rpy="0 0 0" xyz="0.05955 0 0.3"/>
+    <origin rpy="0 0 0" xyz="0.060 0 0.4"/>
     <parent link="$(arg robot_name)/upper_arm_link"/>
-    <child link="$(arg robot_name)/upper_forearm_link"/>
+    <child link="$(arg robot_name)/forearm_link"/>
     <dynamics friction="0.1"/>
   </joint>
@@ -135,59 +135,22 @@
     </actuator>
   </transmission>
-  <link name="$(arg robot_name)/upper_forearm_link">
-    <visual>
-      <origin rpy="0 0 0" xyz="0 0 0"/>
-      <geometry>
-        <mesh filename="package://interbotix_xsarm_descriptions/meshes/vx300s_meshes/vx300s_4_upper_forearm.stl" scale="0.001 0.001 0.001"/>
-      </geometry>
-      <material name="interbotix_black"/>
-    </visual>
-    <collision>
-      <origin rpy="0 0 0" xyz="0 0 0"/>
-      <geometry>
-        <mesh filename="package://interbotix_xsarm_descriptions/meshes/vx300s_meshes/vx300s_4_upper_forearm.stl" scale="0.001 0.001 0.001"/>
-      </geometry>
-    </collision>
-    <inertial>
-      <origin rpy="0 0 0" xyz="0.105723 0 0"/>
-      <mass value="0.322228" />
-      <inertia ixx="0.0001524000" iyy="0.0013420000" izz="0.0014410000" ixy="-0.0000188300" ixz="-0.0000084064" iyz="0.0000012564" />
-    </inertial>
-  </link>
-  <joint name="forearm_roll" type="revolute">
-    <axis xyz="1 0 0"/>
-    <limit effort="2" lower="${-pi + pi_offset}" upper="${pi - pi_offset}" velocity="${pi}"/>
-    <origin rpy="0 0 0" xyz="0.2 0 0"/>
-    <parent link="$(arg robot_name)/upper_forearm_link"/>
-    <child link="$(arg robot_name)/lower_forearm_link"/>
-    <dynamics friction="0.1"/>
-  </joint>
-  <transmission name="trans_forearm_roll">
-    <type>transmission_interface/SimpleTransmission</type>
-    <joint name="forearm_roll">
-      <hardwareInterface>hardware_interface/EffortJointInterface</hardwareInterface>
-    </joint>
-    <actuator name="forearm_roll_motor">
-      <mechanicalReduction>1</mechanicalReduction>
-    </actuator>
-  </transmission>
-  <link name="$(arg robot_name)/lower_forearm_link">
-    <visual>
-      <origin rpy="${pi} 0 0" xyz="0 0 0"/>
-      <geometry>
-        <mesh filename="package://interbotix_xsarm_descriptions/meshes/vx300s_meshes/vx300s_5_lower_forearm.stl" scale="0.001 0.001 0.001"/>
-      </geometry>
-      <material name="interbotix_black"/>
-    </visual>
-    <collision>
-      <origin rpy="${pi} 0 0" xyz="0 0 0"/>
-      <geometry>
-        <mesh filename="package://interbotix_xsarm_descriptions/meshes/vx300s_meshes/vx300s_5_lower_forearm.stl" scale="0.001 0.001 0.001"/>
-      </geometry>
-    </collision>
-    <inertial>
-      <origin rpy="${pi} 0 0" xyz="0.0513477000 0.0068046200 0"/>
-      <mass value="0.414823" />
-      <inertia ixx="0.0001753000" iyy="0.0005269000" izz="0.0005911000" ixy="-0.0000852800" ixz="0" iyz="0" />
+  <link name="$(arg robot_name)/forearm_link">
+    <visual>
+      <origin rpy="0 0 ${pi/2}" xyz="0.285 0.003 -0.035"/>
+      <geometry>
+        <mesh filename="package://interbotix_xsarm_descriptions/meshes/lucasrobot_meshes/lucasrobot_4_forearm.stl" scale="0.001 0.001 0.001"/>
+      </geometry>
+      <material name="interbotix_black"/>
+    </visual>
+    <collision>
+      <origin rpy="0 0 ${pi/2}" xyz="0 0 0"/>
+      <geometry>
+        <mesh filename="package://interbotix_xsarm_descriptions/meshes/lucasrobot_meshes/lucasrobot_4_forearm.stl" scale="0.001 0.001 0.001"/>
+      </geometry>
+    </collision>
+    <inertial>
+      <origin rpy="0 0 ${pi/2}" xyz="0.1812650000 -0.0002065037 0.0000000000"/>
+      <mass value="0.544659" />
+      <inertia ixx="0.0054470000" iyy="0.0002267000" izz="0.0055740000" ixy="-0.0000119800" ixz="0.0000000000" iyz="0.0000000000" />
     </inertial>
   </link>
@@ -195,6 +158,6 @@
     <axis xyz="0 1 0"/>
     <limit effort="5" lower="${radians(-107)}" upper="${radians(128)}" velocity="${pi}"/>
-    <origin rpy="0 0 0" xyz="0.1 0 0"/>
-    <parent link="$(arg robot_name)/lower_forearm_link"/>
+    <origin rpy="0 0 0" xyz="0.434 0 -0.003"/>
+    <parent link="$(arg robot_name)/forearm_link"/>
     <child link="$(arg robot_name)/wrist_link"/>
     <dynamics friction="0.1"/>
@@ -211,14 +174,14 @@
   <link name="$(arg robot_name)/wrist_link">
     <visual>
+      <origin rpy="0 0 ${pi/2}" xyz="0.044 0 -0.050"/>
+      <geometry>
+        <mesh filename="package://interbotix_xsarm_descriptions/meshes/lucasrobot_meshes/lucasrobot_5_wrist.stl" scale="0.001 0.001 0.001"/>
+      </geometry>
+      <material name="interbotix_black"/>
+    </visual>
+    <collision>
       <origin rpy="0 0 ${pi/2}" xyz="0 0 0"/>
       <geometry>
-        <mesh filename="package://interbotix_xsarm_descriptions/meshes/vx300s_meshes/vx300s_6_wrist.stl" scale="0.001 0.001 0.001"/>
-      </geometry>
-      <material name="interbotix_black"/>
-    </visual>
-    <collision>
-      <origin rpy="0 0 ${pi/2}" xyz="0 0 0"/>
-      <geometry>
-        <mesh filename="package://interbotix_xsarm_descriptions/meshes/vx300s_meshes/vx300s_6_wrist.stl" scale="0.001 0.001 0.001"/>
+        <mesh filename="package://interbotix_xsarm_descriptions/meshes/lucasrobot_meshes/lucasrobot_5_wrist.stl" scale="0.001 0.001 0.001"/>
       </geometry>
     </collision>
@@ -232,5 +195,5 @@
     <axis xyz="1 0 0"/>
     <limit effort="1" lower="${-pi + pi_offset}" upper="${pi - pi_offset}" velocity="${pi}"/>
-    <origin rpy="0 0 0" xyz="0.069744 0 0"/>
+    <origin rpy="0 0 0" xyz="0.086 0 0"/>
     <parent link="$(arg robot_name)/wrist_link"/>
     <child link="$(arg robot_name)/gripper_link"/>
@@ -248,14 +211,14 @@
   <link name="$(arg robot_name)/gripper_link">
     <visual>
+      <origin rpy="0 ${pi/2} ${pi/2}" xyz="0.02 -0.05 -0.005"/>
+      <geometry>
+        <mesh filename="package://interbotix_xsarm_descriptions/meshes/lucasrobot_meshes/lucasrobot_6_gripper.stl" scale="0.001 0.001 0.001"/>
+      </geometry>
+      <material name="interbotix_black"/>
+    </visual>
+    <collision>
       <origin rpy="0 0 ${pi/2}" xyz="-0.02 0 0"/>
       <geometry>
-        <mesh filename="package://interbotix_xsarm_descriptions/meshes/vx300s_meshes/vx300s_7_gripper.stl" scale="0.001 0.001 0.001"/>
-      </geometry>
-      <material name="interbotix_black"/>
-    </visual>
-    <collision>
-      <origin rpy="0 0 ${pi/2}" xyz="-0.02 0 0"/>
-      <geometry>
-        <mesh filename="package://interbotix_xsarm_descriptions/meshes/vx300s_meshes/vx300s_7_gripper.stl" scale="0.001 0.001 0.001"/>
+        <mesh filename="package://interbotix_xsarm_descriptions/meshes/lucasrobot_meshes/lucasrobot_6_gripper.stl" scale="0.001 0.001 0.001"/>
       </geometry>
     </collision>
@@ -268,5 +231,5 @@
   <joint name="ee_arm" type="fixed">
     <axis xyz="1 0 0"/>
-    <origin rpy="0 0 0" xyz="0.042825 0 0"/>
+    <origin rpy="0 0 0" xyz="0.065 0 -0.005"/>
     <parent link="$(arg robot_name)/gripper_link"/>
     <child link="$(arg robot_name)/ee_arm_link"/>
@@ -297,14 +260,14 @@
   <link name="$(arg robot_name)/gripper_prop_link">
     <visual>
+      <origin rpy="0 0 ${pi/2}" xyz="-0.01 0.001 -0.028"/>
+      <geometry>
+        <mesh filename="package://interbotix_xsarm_descriptions/meshes/lucasrobot_meshes/lucasrobot_7_gripper_prop.stl" scale="0.001 0.001 0.001"/>
+      </geometry>
+      <material name="interbotix_black"/>
+    </visual>
+    <collision>
       <origin rpy="0 0 ${pi/2}" xyz="-0.0685 0 0"/>
       <geometry>
-        <mesh filename="package://interbotix_xsarm_descriptions/meshes/vx300s_meshes/vx300s_8_gripper_prop.stl" scale="0.001 0.001 0.001"/>
-      </geometry>
-      <material name="interbotix_black"/>
-    </visual>
-    <collision>
-      <origin rpy="0 0 ${pi/2}" xyz="-0.0685 0 0"/>
-      <geometry>
-        <mesh filename="package://interbotix_xsarm_descriptions/meshes/vx300s_meshes/vx300s_8_gripper_prop.stl" scale="0.001 0.001 0.001"/>
+        <mesh filename="package://interbotix_xsarm_descriptions/meshes/lucasrobot_meshes/lucasrobot_7_gripper_prop.stl" scale="0.001 0.001 0.001"/>
       </geometry>
     </collision>
@@ -327,5 +290,5 @@
         <origin rpy="0 0 0" xyz="0 0 0"/>
         <geometry>
-          <mesh filename="package://interbotix_xsarm_descriptions/meshes/vx300s_meshes/vx300s_11_ar_tag.stl" scale="0.001 0.001 0.001"/>
+          <mesh filename="package://interbotix_xsarm_descriptions/meshes/lucasrobot_meshes/lucasrobot_10_ar_tag.stl" scale="0.001 0.001 0.001"/>
         </geometry>
         <material name="interbotix_black"/>
@@ -334,5 +297,5 @@
         <origin rpy="0 0 0" xyz="0 0 0"/>
         <geometry>
-          <mesh filename="package://interbotix_xsarm_descriptions/meshes/vx300s_meshes/vx300s_11_ar_tag.stl" scale="0.001 0.001 0.001"/>
+          <mesh filename="package://interbotix_xsarm_descriptions/meshes/lucasrobot_meshes/lucasrobot_10_ar_tag.stl" scale="0.001 0.001 0.001"/>
         </geometry>
       </collision>
@@ -354,7 +317,7 @@
     <link name="$(arg robot_name)/gripper_bar_link">
       <visual>
-        <origin rpy="0 0 ${pi/2}" xyz="-0.063 0 0"/>
+        <origin rpy="0 0 ${pi/2}" xyz="0.02 0 -0.02"/>
         <geometry>
-          <mesh filename="package://interbotix_xsarm_descriptions/meshes/vx300s_meshes/vx300s_9_gripper_bar.stl" scale="0.001 0.001 0.001"/>
+          <mesh filename="package://interbotix_xsarm_descriptions/meshes/lucasrobot_meshes/lucasrobot_8_gripper_bar.stl" scale="0.001 0.001 0.001"/>
         </geometry>
         <material name="interbotix_black"/>
@@ -363,5 +326,5 @@
         <origin rpy="0 0 ${pi/2}" xyz="-0.063 0 0"/>
         <geometry>
-          <mesh filename="package://interbotix_xsarm_descriptions/meshes/vx300s_meshes/vx300s_9_gripper_bar.stl" scale="0.001 0.001 0.001"/>
+          <mesh filename="package://interbotix_xsarm_descriptions/meshes/lucasrobot_meshes/lucasrobot_8_gripper_bar.stl" scale="0.001 0.001 0.001"/>
         </geometry>
       </collision>
@@ -388,5 +351,5 @@
       <joint name="left_finger" type="prismatic">
         <axis xyz="0 1 0"/>
-        <limit effort="5" lower="0.021" upper="0.057" velocity="1"/>
+        <limit effort="5" lower="0.015" upper="0.04" velocity="1"/>
         <origin rpy="0 0 0" xyz="0 0 0"/>
         <parent link="$(arg robot_name)/fingers_link"/>
@@ -405,25 +368,25 @@
       <link name="$(arg robot_name)/left_finger_link">
         <visual>
-          <origin rpy="${pi/2} ${-pi} ${pi/2}" xyz="-0.0404 -0.0575 0"/>
+          <origin rpy="${-pi/2} 0 ${-pi/2}" xyz="0.035 0.005 0 "/>
           <geometry>
-            <mesh filename="package://interbotix_xsarm_descriptions/meshes/vx300s_meshes/vx300s_10_gripper_finger.stl" scale="0.001 0.001 0.001"/>
+            <mesh filename="package://interbotix_xsarm_descriptions/meshes/lucasrobot_meshes/lucasrobot_9_gripper_finger.stl" scale="0.001 0.001 0.001"/>
           </geometry>
           <material name="interbotix_black"/>
         </visual>
         <collision>
-          <origin rpy="${pi/2} ${-pi} ${pi/2}" xyz="-0.0404 -0.0575 0"/>
+          <origin rpy="${-pi/2} 0 ${-pi/2}" xyz="0.0404 0.0575 0 "/>
           <geometry>
-            <mesh filename="package://interbotix_xsarm_descriptions/meshes/vx300s_meshes/vx300s_10_gripper_finger.stl" scale="0.001 0.001 0.001"/>
+            <mesh filename="package://interbotix_xsarm_descriptions/meshes/lucasrobot_meshes/lucasrobot_9_gripper_finger.stl" scale="0.001 0.001 0.001"/>
           </geometry>
         </collision>
         <inertial>
-          <origin rpy="${pi} ${pi} ${pi/2}" xyz="0.0173440000 -0.0060692000 0.0000000000"/>
+          <origin rpy="0 ${pi} ${pi/2}" xyz="0.0173440000 0.0060692000  0.0000000000"/>
           <mass value="0.034796" />
-          <inertia ixx="0.0000243300" iyy="0.0000125500" izz="0.0000141700" ixy="-0.0000024004" ixz="0.0000000000" iyz="0.0000000000" />
+          <inertia ixx="0.0000243300" iyy="0.0000125500" izz="0.0000141700" ixy="0.0000024001" ixz="0.0000000000" iyz="0.0000000000" />
         </inertial>
       </link>
       <joint name="right_finger" type="prismatic">
         <axis xyz="0 1 0"/>
-        <limit effort="5" lower="-0.057" upper="-0.021" velocity="1"/>
+        <limit effort="5" lower="-0.04" upper="-0.015" velocity="1"/>
         <origin rpy="0 0 0" xyz="0 0 0"/>
         <parent link="$(arg robot_name)/fingers_link"/>
@@ -445,20 +408,20 @@
       <link name="$(arg robot_name)/right_finger_link">
         <visual>
-          <origin rpy="${-pi/2} ${pi} ${-pi/2}" xyz="-0.0404 0.0575 0 "/>
+          <origin rpy="${pi/2} 0 ${pi/2}" xyz="0.035 -0.005 0"/>
           <geometry>
-            <mesh filename="package://interbotix_xsarm_descriptions/meshes/vx300s_meshes/vx300s_10_gripper_finger.stl" scale="0.001 0.001 0.001"/>
+            <mesh filename="package://interbotix_xsarm_descriptions/meshes/lucasrobot_meshes/lucasrobot_9_gripper_finger.stl" scale="0.001 0.001 0.001"/>
           </geometry>
           <material name="interbotix_black"/>
         </visual>
         <collision>
-          <origin rpy="${-pi/2} ${pi} ${-pi/2}" xyz="-0.0404 0.0575 0 "/>
+          <origin rpy="${pi/2} 0 ${pi/2}" xyz="-0.0404 -0.0575 0"/>
           <geometry>
-            <mesh filename="package://interbotix_xsarm_descriptions/meshes/vx300s_meshes/vx300s_10_gripper_finger.stl" scale="0.001 0.001 0.001"/>
+            <mesh filename="package://interbotix_xsarm_descriptions/meshes/lucasrobot_meshes/lucasrobot_9_gripper_finger.stl" scale="0.001 0.001 0.001"/>
           </geometry>
         </collision>
         <inertial>
-          <origin rpy="0 ${pi} ${pi/2}" xyz="0.0173440000 0.0060692000  0.0000000000"/>
+          <origin rpy="${pi} ${pi} ${pi/2}" xyz="0.0173440000 -0.0060692000 0.0000000000"/>
           <mass value="0.034796" />
-          <inertia ixx="0.0000243300" iyy="0.0000125500" izz="0.0000141700" ixy="0.0000024001" ixz="0.0000000000" iyz="0.0000000000" />
+          <inertia ixx="0.0000243300" iyy="0.0000125500" izz="0.0000141700" ixy="-0.0000024004" ixz="0.0000000000" iyz="0.0000000000" />
         </inertial>
       </link>
